Commit message: tfが同じ名前であったのと、Pathがでるように修正

File: traj_follow_plotter/meshes/zx200_video.xacro (robot description, xacro)
@@ -1,12 +1,17 @@
 <?xml version="1.0"?>
 <robot name="zx200" xmlns:xacro="http://www.ros.org/wiki/xacro">
+<!-- プレフィックス用の引数（デフォルトは空） -->
+<xacro:arg name="prefix" default="" />
+<xacro:property name="prefix" value="$(arg prefix)" />
+<!-- ロボット名もプレフィックス付き -->
+<xacro:property name="robot_name" value="${prefix}zx200" />
 <!-- Used for fixing robot to Gazebo 'base_link' -->
-<link name="base_link"/>
-<joint name="base_joint" type="fixed">
-<parent link="base_link"/>
-<child link="track_link"/>
+<link name="${prefix}base_link"/>
+<joint name="${prefix}base_joint" type="fixed">
+<parent link="${prefix}base_link"/>
+<child link="${prefix}track_link"/>
 </joint>
 <!-- Base Link -->
-<link name="track_link">
+<link name="${prefix}track_link">
 <visual>
 <geometry>
@@ -26,11 +31,11 @@
 </link>
 <!-- body axis -->
-<joint name="swing_joint" type="continuous">
+<joint name="${prefix}swing_joint" type="continuous">
 <origin xyz="0.10787 -0.034301 1.1206"/>
 <axis xyz="0 0 1"/>
-<parent link="track_link"/>
-<child link="body_link"/>
+<parent link="${prefix}track_link"/>
+<child link="${prefix}body_link"/>
 </joint>
-<link name="body_link">
+<link name="${prefix}body_link">
 <visual>
 <origin xyz="0 0 0"/>
@@ -52,12 +57,12 @@
 </link>
 <!-- boom axis -->
-<joint name="boom_joint" type="revolute">
+<joint name="${prefix}boom_joint" type="revolute">
 <origin rpy="0 0.559505 0" xyz="0.22767 -0.040187 0.83669"/>
 <axis xyz="0 1 0"/>
-<parent link="body_link"/>
-<child link="boom_link"/>
+<parent link="${prefix}body_link"/>
+<child link="${prefix}boom_link"/>
 <limit lower="-1.137" upper="-0.1" effort="500" velocity="6.159937255"/>
 </joint>
-<link name="boom_link">
+<link name="${prefix}boom_link">
 <visual>
 <origin xyz="0 0 0"/>
@@ -78,12 +83,12 @@
 </inertial>
 </link>
-<joint name="arm_joint" type="revolute">
+<joint name="${prefix}arm_joint" type="revolute">
 <origin rpy="0 0.296258 0" xyz="4.7878 0.010957 2.9959"/>
 <axis xyz="0 1 0"/>
-<parent link="boom_link"/>
-<child link="arm_link"/>
+<parent link="${prefix}boom_link"/>
+<child link="${prefix}arm_link"/>
 <limit lower="0.594" upper="2.531" effort="500" velocity="6.159937255"/>
 </joint>
-<link name="arm_link">
+<link name="${prefix}arm_link">
 <visual>
 <origin xyz="0 0 0"/>
@@ -105,12 +110,12 @@
 </link>
 <!-- bucket axis -->
-<joint name="bucket_joint" type="revolute">
+<joint name="${prefix}bucket_joint" type="revolute">
 <origin rpy="0 -0.160621 0" xyz="1.8954 -0.023546 2.1809"/>
 <axis xyz="0 1 0"/>
-<parent link="arm_link"/>
-<child link="bucket_link"/>
+<parent link="${prefix}arm_link"/>
+<child link="${prefix}bucket_link"/>
 <limit lower="-0.622" upper="2.372" effort="50000" velocity="6.159937255"/>
 </joint>
-<link name="bucket_link">
+<link name="${prefix}bucket_link">
 <visual>
 <origin xyz="0 0 0"/>
@@ -131,5 +136,5 @@
 </inertial>
 </link>
-<link name="bucket_end_link">
+<link name="${prefix}bucket_end_link">
 <visual>
 <origin xyz="0 0 0" rpy="0 0 0"/>
@@ -144,7 +149,7 @@
 </inertial>
 </link>
-<joint name="bucket_end_joint" type="revolute">
-<parent link="bucket_link"/>
-<child link="bucket_end_link"/>
+<joint name="${prefix}bucket_end_joint" type="revolute">
+<parent link="${prefix}bucket_link"/>
+<child link="${prefix}bucket_end_link"/>
 <axis xyz="1 0 0"/>
 <origin rpy="0 0 0" xyz="1.2 0 1"/>
