Commit message: Update the limits of URDF model

File: traj_follow_plotter/urdf/zx200.urdf (robot description, URDF)
Before this commit: robot zx200, 7 links, 6 joints
Joints:
- joint arm_joint: limit lower=0.594 upper=2.531 effort=500 velocity=6.159937255 -> lower=0.58 upper=2.687 effort=500 velocity=6.159937255
- joint boom_joint: limit lower=-1.137 upper=-0.1 effort=500 velocity=6.159937255 -> lower=-1.13 upper=1.15 effort=500 velocity=6.159937255
